File: Tic-Tac-Toe/Schaltplan/Schaltplan.sch (KiCad schematic (older format))
At the start: 164 parts, among them J1 USB_B, J10 Conn_01x03_Male, J11 Conn_01x03_Male, J12 Conn_01x03_Male, J13 Conn_01x03_Male, J2 Conn_01x01_Male, J3 Conn_01x01_Male, J4 Conn_01x01_Male, J5 Conn_01x03_Male, J6 Conn_01x03_Male, J7 Conn_01x03_Male, J8 Conn_01x03_Male, J9 Conn_01x03_Male, Q1 BC337, Q2 BC337, Q3 BC337, SW10 SW_Push_Dual, SW11 SW_Push_Dual, SW12 SW_Push_Dual, SW2 SW_Push_Dual, SW3 SW_Push_Dual, SW4 SW_Push_Dual, SW5 SW_Push_Dual, SW6 SW_Push_Dual, SW7 SW_Push_Dual, SW8 SW_Push_Dual, SW9 SW_Push_Dual, U1 74HC595, U2 74HC595, U3 74HC595, U4 74HC595, U5 74HC595

Commit message: Footprints zum Tic-Tac-Toe zugeordnet
Connections:
- net at A1.5 (D2), SW8.1, SW8.3: now also R51.1
- net at R50.1, SW8.2, SW8.4: no longer R51.1
Other:
- moved on the sheet: R51
Changed lines of the file:
@@
 L power:GND #PWR07
 U 1 1 5EA9A1D6
-P 2700 6100
-F 0 "#PWR07" H 2700 5850 50  0001 C CNN
-F 1 "GND" H 2700 5950 50  0000 C CNN
-F 2 "" H 2700 6100 50  0001 C CNN
-F 3 "" H 2700 6100 50  0001 C CNN
-	1    2700 6100
+P 3700 6100
+F 0 "#PWR07" H 3700 5850 50  0001 C CNN
+F 1 "GND" H 3700 5950 50  0000 C CNN
+F 2 "" H 3700 6100 50  0001 C CNN
+F 3 "" H 3700 6100 50  0001 C CNN
+	1    3700 6100
 	-1   0    0    -1
 $EndComp
@@
 L Device:R R51
 U 1 1 5EA9AAFC
-P 2850 6100
-F 0 "R51" V 2950 6050 50  0000 L CNN
-F 1 "1K" V 2850 6050 50  0000 L CNN
-F 2 "" V 2780 6100 50  0001 C CNN
-F 3 "~" H 2850 6100 50  0001 C CNN
-	1    2850 6100
-	0    1    1    0
+P 3550 6100
+F 0 "R51" V 3650 6050 50  0000 L CNN
+F 1 "1K" V 3550 6050 50  0000 L CNN
+F 2 "" V 3480 6100 50  0001 C CNN
+F 3 "~" H 3550 6100 50  0001 C CNN
+	1    3550 6100
+	0    -1   -1   0
 $EndComp
 $Comp
@@
 Massen>Trennen_und_Dioden
 Connection ~ 3000 5900
-Connection ~ 3000 6100
 $Comp
 L Device:LED D35
