File: Tic-Tac-Toe/Schaltplan_Platine/Schaltplan.kicad_pcb (KiCad board)
At the start: 2 copper layers, 137 parts, among them J1 USB_B, J10 Conn_01x03_Male, J11 Conn_01x03_Male, J12 Conn_01x03_Male, J13 Conn_01x03_Male, J2 Conn_01x01_Male, J3 Conn_01x01_Male, J4 Conn_01x01_Male, J5 Conn_01x03_Male, J6 Conn_01x03_Male, J7 Conn_01x03_Male, J8 Conn_01x03_Male, J9 Conn_01x03_Male, Q1 BC337, Q2 BC337, Q3 BC337, SW10 SW_Push_Dual, SW11 SW_Push_Dual, SW12 SW_Push_Dual, SW2 SW_Push_Dual, SW3 SW_Push_Dual, SW4 SW_Push_Dual, SW5 SW_Push_Dual, SW6 SW_Push_Dual, SW7 SW_Push_Dual, SW8 SW_Push_Dual, SW9 SW_Push_Dual, U1 74HC595, U2 74HC595, U3 74HC595, U4 74HC595, U5 74HC595

Commit message: Schaltplan Update
Parts:
- moved A1 203.2 mm to (-138.1, 63.8)
- moved D30 203.2 mm to (-31.2, 90.0)
- moved D32 203.2 mm to (-62.3, 124.3)
- moved D33 203.2 mm to (-38.5, 98.8)
- moved D34 203.2 mm to (-31.2, 85.4)
- moved D37 203.2 mm to (-62.3, 119.7)
- moved J2 203.2 mm to (-51.7, 112.8)
- moved R13 203.2 mm to (-61.3, 64.3)
- moved R33 203.2 mm to (-61.3, 70.4)
- moved R37 203.2 mm to (-61.3, 67.3)
- moved R40 203.2 mm to (-61.3, 73.4)
- moved R44 203.2 mm to (-61.3, 76.5)
- moved R51 203.2 mm to (-63.3, 82.6)
- moved R59 203.2 mm to (-63.3, 85.6)
- moved R68 203.2 mm to (-32.0, 61.2)
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