File: Tic-Tac-Toe/Schaltplan_Platine/Schaltplan.sch (KiCad schematic (older format))
At the start: 164 parts, among them J1 USB_B, J10 Conn_01x03_Male, J11 Conn_01x03_Male, J12 Conn_01x03_Male, J13 Conn_01x03_Male, J2 Conn_01x01_Male, J3 Conn_01x01_Male, J4 Conn_01x01_Male, J5 Conn_01x03_Male, J6 Conn_01x03_Male, J7 Conn_01x03_Male, J8 Conn_01x03_Male, J9 Conn_01x03_Male, Q1 BC337, Q2 BC337, Q3 BC337, SW10 SW_Push_Dual, SW11 SW_Push_Dual, SW12 SW_Push_Dual, SW2 SW_Push_Dual, SW3 SW_Push_Dual, SW4 SW_Push_Dual, SW5 SW_Push_Dual, SW6 SW_Push_Dual, SW7 SW_Push_Dual, SW8 SW_Push_Dual, SW9 SW_Push_Dual, U1 74HC595, U2 74HC595, U3 74HC595, U4 74HC595, U5 74HC595

Commit message: Footprints zum Tic-Tac-Toe zugeordnet
Parts:
- removed D1, D10, D11, D12, D13, D14, D15, D16, D17, D18, D19, D2, D20, D21, D22, D23, D24, D25, D26, D27, D3, D4, D5, D6, D7, D8, D9: LED_CRGB, symbol Device:LED_CRGB
- C1, C2: footprint (none) -> Capacitor_THT:C_Disc_D4.7mm_W2.5mm_P5.00mm
- D28, D29, D30, D31, D32, D33, D34, D35, D37, D38, D39: footprint (none) -> LED_THT:LED_D3.0mm
- D36: footprint (none) -> LED_THT:LED_D5.0mm-4_RGB
- J1: footprint (none) -> Connector_USB:USB_B_OST_USB-B1HSxx_Horizontal
- J10, J11, J12, J13, J5, J6, J7, J8, J9: footprint (none) -> Connector_PinHeader_2.54mm:PinHeader_1x03_P2.54mm_Vertical
- J2, J3, J4: footprint (none) -> Connector_PinHeader_2.54mm:PinHeader_1x01_P2.54mm_Vertical
- R1, R10, R11, R12, R13, R14, R15, R16, R17, R18, R19, R2, R20, R21, R22, R23, R24, R25, R26, R27, R28, R29, R3, R30, R31, R32, R33, R34, R35, R36, R37, R38, R39, R4, R40, R41, R42, R43, R44, R45, R46, R47, R48, R49, R5, R50, R51, R52, R53, R54, R55, R56, R57, R58, R59, R6, R60, R61, R62, R63, R64, R65, R66, R67, R68, R69, R7, R70, R71, R72, R73, R74, R75, R76, R77, R78, R79, R8, R80, R81, R82, R83, R84, R85, R86, R87, R88, R89, R9: footprint (none) -> Resistor_THT:R_Axial_DIN0207_L6.3mm_D2.5mm_P7.62mm_Horizontal
- RV1: footprint (none) -> Potentiometer_THT:Potentiometer_Alps_RK163_Single_Horizontal
- SW10, SW11, SW12, SW2, SW3, SW4, SW5, SW6, SW7, SW8, SW9: footprint (none) -> Button_Switch_THT:SW_TH_Tactile_Omron_B3F-10xx
- U1, U2, U3, U4, U5: footprint (none) -> Package_DIP:DIP-16_W7.62mm
Connections:
- net at A1.5 (D2), SW8.1, SW8.3: now also R51.1
- net at R50.1, SW8.2, SW8.4: no longer R51.1
Other:
- note added: "The LEDs aren't present on the PCB"
- note removed: "Note:\nPin_Headers are used only as dummy objects for the LED Conectors\nbecause the LEDs aren't placed on the PCB"
- moved on the sheet: J3, J4, R51

Commit message: Schaltplan Update
Changed lines of the file:
@@
 P 8200 3250
 F 0 "J4" V 8260 3290 50  0000 L CNN
-F 1 "Conn_01x01_Male" V 8351 3290 50  0000 L CNN
+F 1 "Conn_01x01_Male" H 8200 3450 50  0000 L CNN
 F 2 "Connector_PinHeader_2.54mm:PinHeader_1x01_P2.54mm_Vertical" H 8200 3250 50  0001 C CNN
 F 3 "~" H 8200 3250 50  0001 C CNN
@@
 P 8800 3400
 F 0 "J5" V 8860 3540 50  0000 L CNN
-F 1 "Conn_01x03_Male" V 8951 3540 50  0000 L CNN
+F 1 "Conn_01x03_Male" H 8700 3700 50  0000 L CNN
 F 2 "Connector_PinHeader_2.54mm:PinHeader_1x03_P2.54mm_Vertical" H 8800 3400 50  0001 C CNN
 F 3 "~" H 8800 3400 50  0001 C CNN
@@
 P 9650 3400
 F 0 "J6" V 9710 3540 50  0000 L CNN
-F 1 "Conn_01x03_Male" V 9801 3540 50  0000 L CNN
+F 1 "Conn_01x03_Male" H 9650 3700 50  0000 L CNN
 F 2 "Connector_PinHeader_2.54mm:PinHeader_1x03_P2.54mm_Vertical" H 9650 3400 50  0001 C CNN
 F 3 "~" H 9650 3400 50  0001 C CNN
@@
 P 10500 3400
 F 0 "J7" V 10560 3540 50  0000 L CNN
-F 1 "Conn_01x03_Male" V 10651 3540 50  0000 L CNN
+F 1 "Conn_01x03_Male" H 10450 3700 50  0000 L CNN
 F 2 "Connector_PinHeader_2.54mm:PinHeader_1x03_P2.54mm_Vertical" H 10500 3400 50  0001 C CNN
 F 3 "~" H 10500 3400 50  0001 C CNN
@@
 P 11350 3400
 F 0 "J8" V 11410 3540 50  0000 L CNN
-F 1 "Conn_01x03_Male" V 11501 3540 50  0000 L CNN
+F 1 "Conn_01x03_Male" H 11350 3700 50  0000 L CNN
 F 2 "Connector_PinHeader_2.54mm:PinHeader_1x03_P2.54mm_Vertical" H 11350 3400 50  0001 C CNN
 F 3 "~" H 11350 3400 50  0001 C CNN
@@
 P 12200 3400
 F 0 "J9" V 12260 3540 50  0000 L CNN
-F 1 "Conn_01x03_Male" V 12351 3540 50  0000 L CNN
+F 1 "Conn_01x03_Male" H 12200 3700 50  0000 L CNN
 F 2 "Connector_PinHeader_2.54mm:PinHeader_1x03_P2.54mm_Vertical" H 12200 3400 50  0001 C CNN
 F 3 "~" H 12200 3400 50  0001 C CNN
@@
 P 13050 3400
 F 0 "J10" V 13110 3540 50  0000 L CNN
-F 1 "Conn_01x03_Male" V 13201 3540 50  0000 L CNN
+F 1 "Conn_01x03_Male" H 13050 3750 50  0000 L CNN
 F 2 "Connector_PinHeader_2.54mm:PinHeader_1x03_P2.54mm_Vertical" H 13050 3400 50  0001 C CNN
 F 3 "~" H 13050 3400 50  0001 C CNN
@@
 P 13900 3400
 F 0 "J11" V 13960 3540 50  0000 L CNN
-F 1 "Conn_01x03_Male" V 14051 3540 50  0000 L CNN
+F 1 "Conn_01x03_Male" H 13900 3750 50  0000 L CNN
 F 2 "Connector_PinHeader_2.54mm:PinHeader_1x03_P2.54mm_Vertical" H 13900 3400 50  0001 C CNN
 F 3 "~" H 13900 3400 50  0001 C CNN
@@
 P 14750 3400
 F 0 "J12" V 14810 3540 50  0000 L CNN
-F 1 "Conn_01x03_Male" V 14901 3540 50  0000 L CNN
+F 1 "Conn_01x03_Male" H 14750 3750 50  0000 L CNN
 F 2 "Connector_PinHeader_2.54mm:PinHeader_1x03_P2.54mm_Vertical" H 14750 3400 50  0001 C CNN
 F 3 "~" H 14750 3400 50  0001 C CNN
@@
 P 15600 3400
 F 0 "J13" V 15660 3540 50  0000 L CNN
-F 1 "Conn_01x03_Male" V 15751 3540 50  0000 L CNN
+F 1 "Conn_01x03_Male" H 15600 3750 50  0000 L CNN
 F 2 "Connector_PinHeader_2.54mm:PinHeader_1x03_P2.54mm_Vertical" H 15600 3400 50  0001 C CNN
 F 3 "~" H 15600 3400 50  0001 C CNN
